File: rampgen.kicad_pcb (KiCad board)
At the start: 2 copper layers, 100.3 x 57.2 mm, 51 parts, among them J1 RAMP_OUT, J2 1V_OUT, J3 Conn_01x02_Female, Q1 2N7000, Q2 2N3906, Q3 2N3904, Q4 2N7000, Q5 2N7000, U1 NE555P, U2 74AHCT123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

Commit message: Updated.
Parts:
- added R14: 47, Resistor_THT:R_Axial_DIN0207_L6.3mm_D2.5mm_P10.16mm_Horizontal, F.Cu at (41.3, 50.8)
- added R15: 3.3k, Resistor_THT:R_Axial_DIN0207_L6.3mm_D2.5mm_P10.16mm_Horizontal, F.Cu at (56.5, 51.4)
- moved TP2 24.4 mm to (69.8, 69.8)
- moved C6 10.2 mm to (51.4, 38.7), turned to 270 degrees
- moved R8 1.91 mm to (56.5, 38.1), turned to 90 degrees
- moved C3 1.27 mm to (47.0, 43.8)
- moved R9 1.27 mm to (29.2, 41.9)
- moved R2 0.90 mm to (47.6, 26.0)
Connections:
- Q4 pad 3: Net-(C6-Pad1) -> Net-(Q4-Pad3)
- RV1 pad 1: Net-(RV1-Pad1) -> Net-(R7-Pad2)
- RV1 pad 2: Net-(R7-Pad2) -> Net-(R6-Pad1)
- RV1 pad 3: Net-(R6-Pad1) -> Net-(RV1-Pad3)
- RV3 pad 3: Net-(Q3-Pad1) -> Net-(R15-Pad1)
- RV4 pad 1: Net-(RV4-Pad1) -> +5V
- RV4 pad 2: +5V -> Net-(R13-Pad1)
- RV4 pad 3: Net-(R13-Pad1) -> Net-(RV4-Pad3)
Routing:
- net Net-(Q3-Pad1): track 40.0 -> 15.9 mm
- net +5V: track 236.5 -> 213.6 mm
- net Net-(Q1-Pad2): track 33.7 -> 56.3 mm
- net Net-(R15-Pad1): track 0.00 -> 16.8 mm
- net Net-(C6-Pad1): track 40.1 -> 52.8 mm
- net Net-(Q4-Pad3): track 0.00 -> 5.61 mm
- net Net-(R7-Pad2): track 21.2 -> 17.6 mm
- net Net-(R13-Pad1): track 33.0 -> 30.1 mm
- net Net-(R10-Pad1): track 17.0 -> 18.3 mm
- net Net-(Q5-Pad3): track 65.3 -> 64.1 mm
- net GND: track 332.4 -> 333.1 mm
- net Net-(C3-Pad2): track 15.6 -> 14.8 mm
Other:
- board text added: "DIVIDER STATE"
- board text removed: "1V SWITCH"
- board text removed: "DIVIDER INTEGRATOR"

Commit message: Updated.
Parts:
- added TP7: RAMP_OUT, TestPoint:TestPoint_THTPad_2.5x2.5mm_Drill1.2mm, F.Cu at (102.9, 56.5)
- added TP8: 1V_OUT, TestPoint:TestPoint_THTPad_2.5x2.5mm_Drill1.2mm, F.Cu at (16.5, 62.2)
- moved TP6 19.8 mm to (29.2, 47.0)
Routing:
- net Net-(J2-Pad1): track 14.5 -> 28.2 mm
- net Net-(J1-Pad1): track 13.2 -> 20.3 mm
- net Net-(Q5-Pad3): track 64.1 -> 59.8 mm
Changed lines of the file:
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@@
     (thickness 1.6)
     (drawings 22)
-    (tracks 261)
+    (tracks 266)
     (zones 0)
-    (modules 53)
+    (modules 55)
     (nets 33)
   )
@@
     (add_net GND)
   )
+  (module TestPoint:TestPoint_THTPad_2.5x2.5mm_Drill1.2mm (layer F.Cu)
+    (at 16.51 62.23)
+    (descr "THT rectangular pad as test Point, square 2.5mm side length, hole diameter 1.2mm")
+    (tags "test point THT pad rectangle square")
+    (attr virtual)
+    (fp_text reference TP8 (at 0 -2.148) (layer F.SilkS)
+      (effects (font (size 1 1) (thickness 0.15)))
+    )
+    (fp_text value 1V_OUT (at 0 2.25) (layer F.Fab)
+      (effects (font (size 1 1) (thickness 0.15)))
+    )
+    (fp_line (start 1.75 1.75) (end -1.75 1.75) (layer F.CrtYd) (width 0.05))
+    (fp_line (start 1.75 1.75) (end 1.75 -1.75) (layer F.CrtYd) (width 0.05))
+    (fp_line (start -1.75 -1.75) (end -1.75 1.75) (layer F.CrtYd) (width 0.05))
+    (fp_line (start -1.75 -1.75) (end 1.75 -1.75) (layer F.CrtYd) (width 0.05))
+    (fp_line (start -1.45 1.45) (end -1.45 -1.45) (layer F.SilkS) (width 0.12))
+    (fp_line (start 1.45 1.45) (end -1.45 1.45) (layer F.SilkS) (width 0.12))
+    (fp_line (start 1.45 -1.45) (end 1.45 1.45) (layer F.SilkS) (width 0.12))
+    (fp_line (start -1.45 -1.45) (end 1.45 -1.45) (layer F.SilkS) (width 0.12))
+    (fp_text user %R (at 0 -2.15) (layer F.Fab)
+      (effects (font (size 1 1) (thickness 0.15)))
+    )
+    (pad 1 thru_hole rect (at 0 0) (size 2.5 2.5) (drill 1.2) (layers *.Cu *.Mask)
+      (net 6 "Net-(J2-Pad1)"))
+  )
+  (module TestPoint:TestPoint_THTPad_2.5x2.5mm_Drill1.2mm (layer F.Cu)
+    (at 102.87 56.515)
+    (descr "THT rectangular pad as test Point, square 2.5mm side length, hole diameter 1.2mm")
+    (tags "test point THT pad rectangle square")
+    (attr virtual)
+    (fp_text reference TP7 (at 0 -2.148) (layer F.SilkS)
+      (effects (font (size 1 1) (thickness 0.15)))
+    )
+    (fp_text value RAMP_OUT (at 0 2.25) (layer F.Fab)
+      (effects (font (size 1 1) (thickness 0.15)))
+    )
+    (fp_line (start 1.75 1.75) (end -1.75 1.75) (layer F.CrtYd) (width 0.05))
+    (fp_line (start 1.75 1.75) (end 1.75 -1.75) (layer F.CrtYd) (width 0.05))
+    (fp_line (start -1.75 -1.75) (end -1.75 1.75) (layer F.CrtYd) (width 0.05))
+    (fp_line (start -1.75 -1.75) (end 1.75 -1.75) (layer F.CrtYd) (width 0.05))
+    (fp_line (start -1.45 1.45) (end -1.45 -1.45) (layer F.SilkS) (width 0.12))
+    (fp_line (start 1.45 1.45) (end -1.45 1.45) (layer F.SilkS) (width 0.12))
+    (fp_line (start 1.45 -1.45) (end 1.45 1.45) (layer F.SilkS) (width 0.12))
+    (fp_line (start -1.45 -1.45) (end 1.45 -1.45) (layer F.SilkS) (width 0.12))
+    (fp_text user %R (at 0 -2.15) (layer F.Fab)
+      (effects (font (size 1 1) (thickness 0.15)))
+    )
+    (pad 1 thru_hole rect (at 0 0) (size 2.5 2.5) (drill 1.2) (layers *.Cu *.Mask)
+      (net 5 "Net-(J1-Pad1)"))
+  )
   (module Resistor_THT:R_Axial_DIN0207_L6.3mm_D2.5mm_P10.16mm_Horizontal (layer F.Cu)
     (at 56.515 51.435 90)
@@
     )
     (fp_text value 3.3k (at 5.08 2.37 90) (layer F.Fab)
-      (effects (font (size 1 1) (thickness 0.15)))
-    )
-    (fp_text user %R (at 5.08 0 90) (layer F.Fab)
       (effects (font (size 1 1) (thickness 0.15)))
     )
@@
     (fp_line (start 11.21 1.5) (end 11.21 -1.5) (layer F.CrtYd) (width 0.05))
     (fp_line (start 11.21 -1.5) (end -1.05 -1.5) (layer F.CrtYd) (width 0.05))
+    (fp_text user %R (at 5.08 0 90) (layer F.Fab)
+      (effects (font (size 1 1) (thickness 0.15)))
+    )
     (pad 2 thru_hole oval (at 10.16 0 90) (size 1.6 1.6) (drill 0.8) (layers *.Cu *.Mask)
       (net 11 "Net-(Q3-Pad1)"))
@@
     )
     (fp_text value 47 (at 5.08 2.37) (layer F.Fab)
-      (effects (font (size 1 1) (thickness 0.15)))
-    )
-    (fp_text user %R (at 5.08 0) (layer F.Fab)
       (effects (font (size 1 1) (thickness 0.15)))
     )
@@
     (fp_line (start 11.21 1.5) (end 11.21 -1.5) (layer F.CrtYd) (width 0.05))
     (fp_line (start 11.21 -1.5) (end -1.05 -1.5) (layer F.CrtYd) (width 0.05))
+    (fp_text user %R (at 5.08 0) (layer F.Fab)
+      (effects (font (size 1 1) (thickness 0.15)))
+    )
     (pad 2 thru_hole oval (at 10.16 0) (size 1.6 1.6) (drill 0.8) (layers *.Cu *.Mask)
       (net 29 "Net-(Q4-Pad3)"))
@@
   )
   (module TestPoint:TestPoint_THTPad_2.5x2.5mm_Drill1.2mm (layer F.Cu)
-    (at 16.51 62.23)
+    (at 29.21 46.99)
     (descr "THT rectangular pad as test Point, square 2.5mm side length, hole diameter 1.2mm")
     (tags "test point THT pad rectangle square")
@@
   (segment (start 96.84 58.74) (end 97.79 59.69) (width 0.3) (layer F.Cu) (net 5))
   (segment (start 96.84 53.26) (end 96.84 55.96) (width 0.3) (layer F.Cu) (net 5))
+  (segment (start 102.87 56.515) (end 102.87 57.785) (width 0.3) (layer F.Cu) (net 5))
+  (segment (start 100.965 59.69) (end 97.79 59.69) (width 0.3) (layer F.Cu) (net 5))
+  (segment (start 102.87 57.785) (end 100.965 59.69) (width 0.3) (layer F.Cu) (net 5))
   (segment (start 27.625 53.26) (end 27.625 55.96) (width 0.3) (layer F.Cu) (net 6))
-  (segment (start 31.75 66.04) (end 31.75 62.23) (width 0.3) (layer F.Cu) (net 6))
-  (segment (start 27.625 55.96) (end 27.625 58.1) (width 0.3) (layer F.Cu) (net 6))
-  (segment (start 27.625 58.1) (end 27.6225 58.1025) (width 0.3) (layer F.Cu) (net 6))
-  (segment (start 31.75 62.23) (end 27.6225 58.1025) (width 0.3) (layer F.Cu) (net 6))
+  (segment (start 22.78 55.96) (end 16.51 62.23) (width 0.3) (layer F.Cu) (net 6))
+  (segment (start 27.625 55.96) (end 22.78 55.96) (width 0.3) (layer F.Cu) (net 6))
+  (segment (start 27.625 57.47) (end 27.625 55.96) (width 0.3) (layer F.Cu) (net 6))
+  (segment (start 31.75 61.595) (end 27.625 57.47) (width 0.3) (layer F.Cu) (net 6))
+  (segment (start 31.75 66.04) (end 31.75 61.595) (width 0.3) (layer F.Cu) (net 6))
   (segment (start 64.77 50.8) (end 59.69 55.88) (width 0.3) (layer F.Cu) (net 7))
   (segment (start 64.77 49.53) (end 64.77 50.8) (width 0.3) (layer F.Cu) (net 7))
@@
   (segment (start 48.895 57.785) (end 49.53 57.785) (width 0.3) (layer B.Cu) (net 13))
   (segment (start 50.165 58.42) (end 50.165 65.405) (width 0.3) (layer B.Cu) (net 13))
-  (segment (start 16.51 57.15) (end 16.51 62.23) (width 0.3) (layer F.Cu) (net 14))
   (segment (start 19.05 54.61) (end 16.51 57.15) (width 0.3) (layer F.Cu) (net 14))
   (segment (start 19.05 48.895) (end 19.05 54.61) (width 0.3) (layer F.Cu) (net 14))
-  (segment (start 19.05 48.895) (end 35.56 48.895) (width 0.3) (layer F.Cu) (net 14))
   (segment (start 40.64 53.975) (end 40.64 54.61) (width 0.3) (layer F.Cu) (net 14))
   (segment (start 40.64 54.61) (end 40.64 55.88) (width 0.3) (layer F.Cu) (net 14))
   (segment (start 30.875 54.61) (end 29.525 53.26) (width 0.3) (layer F.Cu) (net 14))
-  (segment (start 19.05 40.64) (end 19.05 48.895) (width 0.3) (layer F.Cu) (net 14))
   (segment (start 22.86 36.83) (end 19.05 40.64) (width 0.3) (layer F.Cu) (net 14))
   (segment (start 34.925 54.61) (end 38.1 51.435) (width 0.3) (layer F.Cu) (net 14))
@@
   (segment (start 34.29 54.61) (end 30.875 54.61) (width 0.3) (layer F.Cu) (net 14))
   (segment (start 38.1 51.435) (end 40.64 53.975) (width 0.3) (layer F.Cu) (net 14))
-  (segment (start 35.56 48.895) (end 38.1 51.435) (width 0.3) (layer F.Cu) (net 14))
+  (segment (start 19.05 46.99) (end 29.21 46.99) (width 0.3) (layer F.Cu) (net 14))
+  (segment (start 19.05 40.64) (end 19.05 46.99) (width 0.3) (layer F.Cu) (net 14))
+  (segment (start 19.05 46.99) (end 19.05 48.895) (width 0.3) (layer F.Cu) (net 14))
+  (segment (start 38.1 51.435) (end 33.655 46.99) (width 0.3) (layer F.Cu) (net 14))
+  (segment (start 33.655 46.99) (end 29.21 46.99) (width 0.3) (layer F.Cu) (net 14))
   (segment (start 100.33 38.1) (end 100.33 43.18) (width 0.3) (layer F.Cu) (net 15))
   (segment (start 69.85 35.56) (end 67.31 38.1) (width 0.3) (layer F.Cu) (net 16))
